File: level_shifter_bidirectional_sch.kicad_sch (KiCad schematic)
At the start: 3 parts

Commit message: updated schematic
Changed lines of the file:
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@@
     (stroke (width 0) (type default) (color 0 0 0 0))
+  )
+  (label "I2C level shifter" (at 175.26 110.49 0)
+    (effects (font (size 1.27 1.27)) (justify left bottom))
   )
   (hierarchical_label "3V3_Logic" (shape input) (at 123.19 111.76 180)
