File: sensors.kicad_sch (KiCad schematic)
At the start: 11 parts

Commit message: added hierarchical labels
Connections:
- net +3V3 is gone; now on net VDD: U?.11 (VBCKUP)
Changed lines of the file:
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@@
     (stroke (width 0) (type default) (color 0 0 0 0))
   )
-  (wire (pts (xy 97.79 46.99) (xy 100.33 46.99))
+  (wire (pts (xy 91.44 46.99) (xy 100.33 46.99))
     (stroke (width 0) (type default) (color 0 0 0 0))
   )
@@
     (stroke (width 0) (type default) (color 0 0 0 0))
   )
-  (wire (pts (xy 111.76 54.61) (xy 111.76 55.88))
+  (wire (pts (xy 111.76 54.61) (xy 111.76 58.42))
     (stroke (width 0) (type default) (color 0 0 0 0))
   )
@@
     (stroke (width 0) (type default) (color 0 0 0 0))
   )
+  (polyline (pts (xy 81.28 63.5) (xy 81.28 67.31))
+    (stroke (width 0) (type default) (color 0 0 0 0))
+  )
   (polyline (pts (xy 81.28 74.93) (xy 133.35 74.93))
     (stroke (width 0) (type default) (color 0 0 0 0))
@@
     (stroke (width 0) (type default) (color 0 0 0 0))
   )
-  (polyline (pts (xy 133.35 63.5) (xy 81.28 63.5))
+  (polyline (pts (xy 133.35 63.5) (xy 133.35 67.31))
+    (stroke (width 0) (type default) (color 0 0 0 0))
+  )
+  (polyline (pts (xy 133.35 67.31) (xy 81.28 67.31))
     (stroke (width 0) (type default) (color 0 0 0 0))
   )
@@
     )
   )
-  (global_label "VCC" (shape input) (at 97.79 46.99 180) (fields_autoplaced)
-    (effects (font (size 1.27 1.27)) (justify right))
+  (global_label "VCC" (shape input) (at 95.25 46.99 90) (fields_autoplaced)
+    (effects (font (size 1.27 1.27)) (justify left))
+    (property "Intersheet References" "${INTERSHEET_REFS}" (id 0) (at 95.1706 41.0372 90)
+      (effects (font (size 1.27 1.27)) (justify left) hide)
+    )
+  )
+  (global_label "GND" (shape input) (at 107.95 120.65 90) (fields_autoplaced)
+    (effects (font (size 1.27 1.27)) (justify left))
+    (property "Intersheet References" "${INTERSHEET_REFS}" (id 0) (at -256.54 -58.42 0)
+      (effects (font (size 1.27 1.27)) hide)
+    )
+  )
+  (global_label "VCC" (shape input) (at 107.95 129.54 180) (fields_autoplaced)
+    (effects (font (size 1.27 1.27)) (justify right))
+    (property "Intersheet References" "${INTERSHEET_REFS}" (id 0) (at -256.54 -58.42 0)
+      (effects (font (size 1.27 1.27)) hide)
+    )
+  )
+  (global_label "GND" (shape input) (at 110.49 166.37 270) (fields_autoplaced)
+    (effects (font (size 1.27 1.27)) (justify right))
+    (property "Intersheet References" "${INTERSHEET_REFS}" (id 0) (at -256.54 -58.42 0)
+      (effects (font (size 1.27 1.27)) hide)
+    )
+  )
+  (global_label "GND" (shape input) (at 111.76 57.15 0) (fields_autoplaced)
+    (effects (font (size 1.27 1.27)) (justify left))
+    (property "Intersheet References" "${INTERSHEET_REFS}" (id 0) (at 117.9547 57.0706 0)
+      (effects (font (size 1.27 1.27)) (justify left) hide)
+    )
+  )
+  (global_label "VDD" (shape input) (at 120.65 132.08 0) (fields_autoplaced)
+    (effects (font (size 1.27 1.27)) (justify left))
+    (property "Intersheet References" "${INTERSHEET_REFS}" (id 0) (at 126.6028 132.0006 0)
+      (effects (font (size 1.27 1.27)) (justify left) hide)
+    )
+  )
+  (global_label "VDD" (shape input) (at 123.19 80.01 0) (fields_autoplaced)
+    (effects (font (size 1.27 1.27)) (justify left))
+    (property "Intersheet References" "${INTERSHEET_REFS}" (id 0) (at -162.56 -8.89 0)
+      (effects (font (size 1.27 1.27)) hide)
+    )
+  )
+  (global_label "VDD" (shape input) (at 127 46.99 0) (fields_autoplaced)
+    (effects (font (size 1.27 1.27)) (justify left))
     (property "Intersheet References" "${INTERSHEET_REFS}" (id 0) (at -162.56 -5.08 0)
       (effects (font (size 1.27 1.27)) hide)
     )
   )
-  (global_label "RX" (shape input) (at 97.79 156.21 180) (fields_autoplaced)
-    (effects (font (size 1.27 1.27)) (justify right))
-    (property "Intersheet References" "${INTERSHEET_REFS}" (id 0) (at -256.54 -58.42 0)
-      (effects (font (size 1.27 1.27)) hide)
-    )
-  )
-  (global_label "TX" (shape input) (at 97.79 158.75 180) (fields_autoplaced)
-    (effects (font (size 1.27 1.27)) (justify right))
-    (property "Intersheet References" "${INTERSHEET_REFS}" (id 0) (at -256.54 -58.42 0)
-      (effects (font (size 1.27 1.27)) hide)
-    )
-  )
-  (global_label "GND" (shape input) (at 107.95 120.65 90) (fields_autoplaced)
-    (effects (font (size 1.27 1.27)) (justify left))
-    (property "Intersheet References" "${INTERSHEET_REFS}" (id 0) (at -256.54 -58.42 0)
-      (effects (font (size 1.27 1.27)) hide)
-    )
-  )
-  (global_label "VCC" (shape input) (at 107.95 129.54 180) (fields_autoplaced)
-    (effects (font (size 1.27 1.27)) (justify right))
-    (property "Intersheet References" "${INTERSHEET_REFS}" (id 0) (at -256.54 -58.42 0)
-      (effects (font (size 1.27 1.27)) hide)
-    )
-  )
-  (global_label "GND" (shape input) (at 110.49 166.37 270) (fields_autoplaced)
-    (effects (font (size 1.27 1.27)) (justify right))
-    (property "Intersheet References" "${INTERSHEET_REFS}" (id 0) (at -256.54 -58.42 0)
-      (effects (font (size 1.27 1.27)) hide)
-    )
-  )
-  (global_label "GND" (shape input) (at 111.76 55.88 270) (fields_autoplaced)
-    (effects (font (size 1.27 1.27)) (justify right))
-    (property "Intersheet References" "${INTERSHEET_REFS}" (id 0) (at -162.56 -5.08 0)
-      (effects (font (size 1.27 1.27)) hide)
-    )
-  )
-  (global_label "VDD" (shape input) (at 123.19 80.01 0) (fields_autoplaced)
-    (effects (font (size 1.27 1.27)) (justify left))
-    (property "Intersheet References" "${INTERSHEET_REFS}" (id 0) (at -162.56 -8.89 0)
-      (effects (font (size 1.27 1.27)) hide)
-    )
-  )
-  (global_label "VDD" (shape input) (at 127 46.99 0) (fields_autoplaced)
-    (effects (font (size 1.27 1.27)) (justify left))
-    (property "Intersheet References" "${INTERSHEET_REFS}" (id 0) (at -162.56 -5.08 0)
-      (effects (font (size 1.27 1.27)) hide)
-    )
-  )
   (global_label "GND" (shape input) (at 171.45 92.71 270) (fields_autoplaced)
     (effects (font (size 1.27 1.27)) (justify right))
@@
     )
   )
-  (global_label "SCL" (shape input) (at 176.53 58.42 180) (fields_autoplaced)
+  (global_label "GND" (shape input) (at 193.04 92.71 270) (fields_autoplaced)
     (effects (font (size 1.27 1.27)) (justify right))
     (property "Intersheet References" "${INTERSHEET_REFS}" (id 0) (at -157.48 -3.81 0)
@@
     )
   )
-  (global_label "SDA" (shape input) (at 176.53 60.96 180) (fields_autoplaced)
-    (effects (font (size 1.27 1.27)) (justify right))
+  (global_label "VDD" (shape input) (at 208.28 43.18 0) (fields_autoplaced)
+    (effects (font (size 1.27 1.27)) (justify left))
     (property "Intersheet References" "${INTERSHEET_REFS}" (id 0) (at -157.48 -3.81 0)
       (effects (font (size 1.27 1.27)) hide)
     )
   )
-  (global_label "GND" (shape input) (at 193.04 92.71 270) (fields_autoplaced)
-    (effects (font (size 1.27 1.27)) (justify right))
-    (property "Intersheet References" "${INTERSHEET_REFS}" (id 0) (at -157.48 -3.81 0)
-      (effects (font (size 1.27 1.27)) hide)
-    )
-  )
-  (global_label "VDD" (shape input) (at 208.28 43.18 0) (fields_autoplaced)
-    (effects (font (size 1.27 1.27)) (justify left))
-    (property "Intersheet References" "${INTERSHEET_REFS}" (id 0) (at -157.48 -3.81 0)
-      (effects (font (size 1.27 1.27)) hide)
-    )
-  )
-  (symbol (lib_id "power:+3.3V") (at 120.65 132.08 0) (unit 1)
-    (in_bom yes) (on_board yes)
-    (property "Reference" "#PWR?" (id 0) (at 120.65 135.89 0)
-      (effects (font (size 1.27 1.27)) hide)
-    )
-    (property "Value" "+3.3V" (id 1) (at 121.031 127.6858 0))
-    (property "Footprint" "" (id 2) (at 120.65 132.08 0)
-      (effects (font (size 1.27 1.27)) hide)
-    )
-    (property "Datasheet" "" (id 3) (at 120.65 132.08 0)
-      (effects (font (size 1.27 1.27)) hide)
-    )
-    (pin "1")
+  (hierarchical_label "Vcc" (shape input) (at 91.44 46.99 180)
+    (effects (font (size 1.27 1.27)) (justify right))
+  )
+  (hierarchical_label "RX" (shape input) (at 97.79 156.21 180)
+    (effects (font (size 1.27 1.27)) (justify right))
+  )
+  (hierarchical_label "TX" (shape input) (at 97.79 158.75 180)
+    (effects (font (size 1.27 1.27)) (justify right))
+  )
+  (hierarchical_label "GND" (shape input) (at 111.76 58.42 270)
+    (effects (font (size 1.27 1.27)) (justify right))
+  )
+  (hierarchical_label "SCL" (shape input) (at 176.53 58.42 180)
+    (effects (font (size 1.27 1.27)) (justify right))
+  )
+  (hierarchical_label "SDA" (shape input) (at 176.53 60.96 180)
+    (effects (font (size 1.27 1.27)) (justify right))
   )
   (symbol (lib_id "Device:C") (at 90.17 83.82 180) (unit 1)
@@
   (symbol (lib_id "RF_GPS:RXM-GPS-RM") (at 110.49 151.13 0) (unit 1)
     (in_bom yes) (on_board yes)
-    (property "Reference" "U?" (id 0) (at 124.3076 149.9616 0)
+    (property "Reference" "U?" (id 0) (at 110.3376 152.5016 0)
       (effects (font (size 1.27 1.27)) (justify left))
     )
-    (property "Value" "RXM-GPS-RM" (id 1) (at 124.3076 152.273 0)
+    (property "Value" "RXM-GPS-RM" (id 1) (at 105.2576 156.083 0)
       (effects (font (size 1.27 1.27)) (justify left))
     )

Commit message: updated for winter 2022
Parts:
- gave numbers to parts that had none: 11
Changed lines of the file:
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@@
   (symbol (lib_id "Device:C") (at 90.17 83.82 180) (unit 1)
     (in_bom yes) (on_board yes)
-    (property "Reference" "C?" (id 0) (at 93.98 83.82 90))
+    (property "Reference" "C3" (id 0) (at 93.98 83.82 90))
     (property "Value" "100n" (id 1) (at 86.36 83.82 90))
     (property "Footprint" "Capacitor_SMD:C_0603_1608Metric_Pad1.08x0.95mm_HandSolder" (id 2) (at 89.2048 80.01 0)
@@
   (symbol (lib_id "Device:C") (at 100.33 50.8 180) (unit 1)
     (in_bom yes) (on_board yes)
-    (property "Reference" "C?" (id 0) (at 104.14 50.8 90))
+    (property "Reference" "C4" (id 0) (at 104.14 50.8 90))
     (property "Value" "100n" (id 1) (at 96.52 50.8 90))
     (property "Footprint" "Capacitor_SMD:C_0603_1608Metric_Pad1.08x0.95mm_HandSolder" (id 2) (at 99.3648 46.99 0)
@@
   (symbol (lib_id "Device:C") (at 107.95 83.82 180) (unit 1)
     (in_bom yes) (on_board yes)
-    (property "Reference" "C?" (id 0) (at 111.76 83.82 90))
+    (property "Reference" "C5" (id 0) (at 111.76 83.82 90))
     (property "Value" "100n" (id 1) (at 104.14 83.82 90))
     (property "Footprint" "Capacitor_SMD:C_0603_1608Metric_Pad1.08x0.95mm_HandSolder" (id 2) (at 106.9848 80.01 0)
@@
   (symbol (lib_id "Device:C") (at 107.95 124.46 180) (unit 1)
     (in_bom yes) (on_board yes)
-    (property "Reference" "C?" (id 0) (at 111.76 124.46 90))
+    (property "Reference" "C6" (id 0) (at 111.76 124.46 90))
     (property "Value" "1u" (id 1) (at 104.14 124.46 90))
     (property "Footprint" "Capacitor_SMD:C_0603_1608Metric_Pad1.08x0.95mm_HandSolder" (id 2) (at 106.9848 120.65 0)
@@
   (symbol (lib_id "Device:C") (at 118.11 83.82 180) (unit 1)
     (in_bom yes) (on_board yes)
-    (property "Reference" "C?" (id 0) (at 121.92 83.82 90))
+    (property "Reference" "C7" (id 0) (at 121.92 83.82 90))
     (property "Value" "10u" (id 1) (at 114.3 83.82 90))
     (property "Footprint" "Capacitor_SMD:C_0603_1608Metric_Pad1.08x0.95mm_HandSolder" (id 2) (at 117.1448 80.01 0)
@@
   (symbol (lib_id "Device:C") (at 123.19 50.8 180) (unit 1)
     (in_bom yes) (on_board yes)
-    (property "Reference" "C?" (id 0) (at 127 50.8 90))
+    (property "Reference" "C8" (id 0) (at 127 50.8 90))
     (property "Value" "10u" (id 1) (at 119.38 50.8 90))
     (property "Footprint" "Capacitor_SMD:C_0603_1608Metric_Pad1.08x0.95mm_HandSolder" (id 2) (at 122.2248 46.99 0)
@@
   (symbol (lib_id "Device:C") (at 161.29 87.63 180) (unit 1)
     (in_bom yes) (on_board yes)
-    (property "Reference" "C?" (id 0) (at 165.1 87.63 90))
+    (property "Reference" "C9" (id 0) (at 165.1 87.63 90))
     (property "Value" "10n" (id 1) (at 157.48 87.63 90))
     (property "Footprint" "Capacitor_SMD:C_0603_1608Metric_Pad1.08x0.95mm_HandSolder" (id 2) (at 160.3248 83.82 0)
@@
   (symbol (lib_id "Device:C") (at 171.45 87.63 180) (unit 1)
     (in_bom yes) (on_board yes)
-    (property "Reference" "C?" (id 0) (at 175.26 87.63 90))
+    (property "Reference" "C10" (id 0) (at 175.26 87.63 90))
     (property "Value" "100n" (id 1) (at 167.64 87.63 90))
     (property "Footprint" "Capacitor_SMD:C_0603_1608Metric_Pad1.08x0.95mm_HandSolder" (id 2) (at 170.4848 83.82 0)
@@
   (symbol (lib_id "Regulator_Linear:IFX27001TFV33") (at 111.76 46.99 0) (unit 1)
     (in_bom yes) (on_board yes)
-    (property "Reference" "U?" (id 0) (at 111.76 40.2082 0))
+    (property "Reference" "U3" (id 0) (at 111.76 40.2082 0))
     (property "Value" "IFX27001TFV33" (id 1) (at 111.76 42.5196 0))
     (property "Footprint" "Package_TO_SOT_SMD:TO-252-3_TabPin2" (id 2) (at 111.76 48.26 0)
@@
   (symbol (lib_id "RF_GPS:RXM-GPS-RM") (at 110.49 151.13 0) (unit 1)
     (in_bom yes) (on_board yes)
-    (property "Reference" "U?" (id 0) (at 110.3376 152.5016 0)
+    (property "Reference" "U2" (id 0) (at 110.3376 152.5016 0)
       (effects (font (size 1.27 1.27)) (justify left))
     )
@@
   (symbol (lib_id "Sensor_Motion:LSM9DS1") (at 195.58 68.58 0) (unit 1)
     (in_bom yes) (on_board yes)
-    (property "Reference" "U?" (id 0) (at 195.58 69.85 0))
+    (property "Reference" "U4" (id 0) (at 195.58 69.85 0))
     (property "Value" "LSM9DS1" (id 1) (at 196.85 72.39 0))
     (property "Footprint" "Package_LGA:LGA-24L_3x3.5mm_P0.43mm" (id 2) (at 233.68 49.53 0)
